File: 12-well_plate_light _box/file5E73C4B8.sch (KiCad schematic (older format))
At the start: 0 parts

Commit message: added single well
Parts:
- added C? (x2): 10uF, symbol Device:C_Small
- added C? (x2): 0.1uF, symbol Device:C_Small
- added D? (x7): LED, symbol 12wp-rescue:WURTH_150141BS63140-custom
- added Q?: NTR3C21NZ-Transistor_FET, Package_TO_SOT_SMD:SOT-23, symbol 12wp-rescue:NTR3C21NZ-Transistor_FET
- added R? (x7): R_Small_US, symbol Device:R_Small_US
- added R? (x2): 1k, symbol Device:R_Small_US
- added R? (x2): 10k, symbol Device:R_Small_US
- added U?: LT3080xDD, Package_DFN_QFN:DFN-8-1EP_3x3mm_P0.5mm_EP1.66x2.38mm, symbol Regulator_Linear:LT3080xDD
- added U?: AD5693RxRM, Package_SO:MSOP-10_3x3mm_P0.5mm, symbol Analog_DAC:AD5693RxRM
Connections:
- new net: R?.1, R?.1, R?.1, R?.1, R?.1, R?.1, R?.1, R?.1, U?.1 (OUT), U?.2 (OUT), U?.3 (OUT), U?.9 (OUT)
- new net: R?.1, R?.1, U?.4 (SET)
- new net: R?.2, U?.10 (VOUT)
- new net: D?.1, D?.3, D?.4, R?.2 (x7)
- new net: D?.2, D?.2, D?.2, D?.2, D?.2, D?.2, D?.2, Q?.3 (D)
- new net +3V3: C?.1, C?.1, C?.1, C?.1, R?.2, U?.1 (VDD), U?.2 (VLOGIC), U?.5 (VCONTROL), U?.7 (IN), U?.8 (IN), U?.9 (VREF)
- new net GND: C?.2, C?.2, C?.2, C?.2, Q?.2 (S), R?.2, R?.2, U?.4 (~LDAC), U?.5 (GND), U?.6 (A0)
